File: PCBs/BoilerBot/BoilerBot.kicad_pcb (KiCad board)
At the start: 2 copper layers, 106 x 4.7 mm, 24 parts, among them J1 Screw_Terminal_01x02, J10 Conn_01x03_Male, J2 Screw_Terminal_01x03, J3 Screw_Terminal_01x03, J4 Screw_Terminal_01x02, J5 Conn_01x05_Male, J6 Conn_01x03_Male, J7 Conn_01x03_Male, J8 Screw_Terminal_01x03, J9 Conn_01x04_Male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

Commit message: PCBs ready to order
Parts:
- C3: footprint Capacitor_SMD:C_0805_2012Metric_Pad1.18x1.45mm_HandSolder -> Capacitor_SMD:CP_Elec_6.3x7.7
- K1: footprint Relay_THT:Relay_1P1T_NO_10x24x18.8mm_Panasonic_ADW11xxxxW_THT -> BoilerBot:OMRON_G5PZ-1A
- moved Q2 86.5 mm to (89.5, 72.5), turned to 180 degrees
- moved R3 63.1 mm to (154.5, 54.0)
- moved J6 58.2 mm to (128.0, 63.5)
- moved BZ1 55.9 mm to (116.0, 74.5)
- moved C3 55.1 mm to (153.5, 61.8), turned to 270 degrees
- moved C1 53.5 mm to (135.0, 59.5), turned to 180 degrees
- moved J9 53.2 mm to (155.5, 73.0), turned to 180 degrees
- moved U1 51.9 mm to (140.5, 62.9), turned to 270 degrees
- moved R1 50.9 mm to (150.5, 68.2), turned to 180 degrees
- moved R2 48.6 mm to (147.0, 68.2), turned to 180 degrees
- moved J10 44.8 mm to (136.5, 70.5)
- moved C2 42.6 mm to (154.5, 56.0)
- moved Q1 42.1 mm to (124.0, 78.5), turned to 180 degrees
- moved A1 41.0 mm to (168.9, 52.0)
- moved J7 37.0 mm to (136.5, 77.5)
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Connections:
- A1 pad 11: MOT1 -> DOWN
- A1 pad 12: MOT2 -> TEMP
- A1 pad 7: UP -> MOT1
- A1 pad 8: DOWN -> MOT2
- A1 pad 9: TEMP -> UP
Routing:
- net HEAT: track 0.00 -> 96.9 mm
- net BUZZ: track 0.00 -> 59.1 mm
- net +12V: track 0.00 -> 40.4 mm
- net GND: track 122.3 -> 159.0 mm, vias 0 -> 6
- net ENCA: track 0.00 -> 35.1 mm
- net UP: track 0.00 -> 34.4 mm
- net ENCB: track 0.00 -> 31.3 mm
- net TEMP: track 0.00 -> 31.1 mm
- net DOWN: track 0.00 -> 25.1 mm
- net LA: track 44.5 -> 21.2 mm
- net SCL: track 0.00 -> 17.9 mm
- net MOT2: track 0.00 -> 17.7 mm
- net MOT1: track 0.00 -> 15.3 mm
- net SDA: track 0.00 -> 14.3 mm
- net PB: track 0.00 -> 14.2 mm
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- added copper zone on F.Cu, net +5V
- added copper zone on B.Cu, net GND
Other:
- board size 106 x 4.7 mm -> 100 x 34 mm
- board text added: "12V"
- board text added: "DOWN 5V"
- board text added: "ENC GND"
- board text added: "GND"
- board text added: "L"
- board text added: "LA"
- board text added: "LCD 5V"
- board text added: "MOT-"
- board text added: "N"
- board text added: "TEMP 5V"
- board text added: "UP 5V"

Commit message: gerber files
Other:
- board text added: "SAGE ROBOTS BOILERBOT 1.0"
