File: PCBs/Encoder/Encoder.kicad_pcb (KiCad board)
At the start: 2 copper layers, 15.5 x 25.5 mm, 4 parts, among them J1 Conn_01x05_Male

Commit message: PCBs ready to order
Other:
- board text added: "GND"
